File: debugger2/debugger2.sch (KiCad schematic (older format))
At the start: 63 parts, among them IC1 AT24CS32-SSHM, P1 CONN_01X01, P2 CONN_01X01, P3 USB_OTG, P4 CONN_02X20, P5 CONN_01X02, Q1 Q_PMOS_GSD, Q2 DMMT3906_Dual_PNP, U1 93LC56B, U2 MIC9409x_SC-70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

Commit message: rev 2.1 fixes for UART, JTAG resets, EEPROM packages
* fix UART (FTDI Ch B) RX/TX backwards
* fix GPIO22_TRST floating by connecting to FTDI Ch A. in debugger 1 we pulled up to 3.3V, but this gives us software control of tap reset
* add options to control RPi power (reset) from FTDI Ch A and button. diodes can be left off BOM to disable a source
* add external drain resistor for vbus switch (backpowering from rpi can cause fet drain in the switch to magic smoke)
* add grounding pad for probe clips
* make holes floating so we can use metal standoffs
* make FB1, FB2 be 0805 (not available in 0603)
* make both EEPROMs TSSOP for easier purchasing (but not compatible)
* reroute USB to a shorter path
Parts:
- removed C10: 4.7u, Capacitors_Tantalum_SMD:TantalC_SizeA_EIA-3216_Wave, symbol CP1_Small
- added D4, D5: D_Small, Diodes_SMD:SOD-523, symbol D_Small
- added R19: 10k, Resistors_SMD:R_0603, symbol R_Small
- added SW1: SW_PUSH, Buttons_Switches_SMD:SW_SPST_EVPBF, symbol SW_PUSH
- FB1, FB2: footprint Resistors_SMD:R_0603 -> Resistors_SMD:R_0805
- U1: footprint Housings_SSOP:MSOP-8_3x3mm_Pitch0.65mm -> Housings_SSOP:TSSOP-8_4.4x3mm_Pitch0.65mm
- U6: renamed from IC1; footprint Housings_SOIC:SOIC-8_3.9x4.9mm_Pitch1.27mm -> Housings_SSOP:TSSOP-8_4.4x3mm_Pitch0.65mm
Connections:
- net labels added: ~JTAG_SRST, ~UART_DTR
- wire segments 259 -> 263
- no-connect marks 3 -> 7
Other:
- note added: "Populate diodes for each allowed system reset source.\nWe cannot guarantee the FTDI configuration will use\nopen drain, so diodes prevent accidental shorting."
- moved on the sheet: C22, P1, P2, P5, R16, R17, R18, R6, R7, R8, U6

Commit message: rev 2.1.1 swap usb micro b to SMT version since many board houses can't make the slots
Parts:
- P3: footprint Connect:USB_Micro-B -> debugger2-special:USB_Micro-B_SMT
Changed lines of the file:
@@
 F 0 "P3" H 6325 5575 50  0000 C CNN
 F 1 "USB_OTG" H 6000 5900 50  0000 C CNN
-F 2 "Connect:USB_Micro-B" V 5950 5600 50  0001 C CNN
+F 2 "debugger2-special:USB_Micro-B_SMT" V 5950 5600 50  0001 C CNN
 F 3 "" V 5950 5600 50  0000 C CNN
 	1    6000 5700

Commit message: rev 2.1.2 swap tantalum caps for ceramic, 2:1 aspect vias
Parts:
- C11, C14, C15, C5, C8: footprint Capacitors_Tantalum_SMD:TantalC_SizeA_EIA-3216_Wave -> Capacitors_SMD:C_1206
Changed lines of the file:
@@
 Title "Raspberry Pi Debugger"
 Date ""
-Rev "2.1"
+Rev "2.1.2"
 Comp "Carnegie Mellon University"
 Comment1 "Based on FT2232H Mini Module"
@@
 F 0 "C14" H 3410 2770 50  0000 L CNN
 F 1 "4.7u" H 3410 2620 50  0000 L CNN
-F 2 "Capacitors_Tantalum_SMD:TantalC_SizeA_EIA-3216_Wave" H 3400 2700 50  0001 C CNN
+F 2 "Capacitors_SMD:C_1206" H 3400 2700 50  0001 C CNN
 F 3 "" H 3400 2700 50  0000 C CNN
 	1    3400 2700
@@
 F 0 "C15" H 3810 1770 50  0000 L CNN
 F 1 "4.7u" H 3810 1620 50  0000 L CNN
-F 2 "Capacitors_Tantalum_SMD:TantalC_SizeA_EIA-3216_Wave" H 3800 1700 50  0001 C CNN
+F 2 "Capacitors_SMD:C_1206" H 3800 1700 50  0001 C CNN
 F 3 "" H 3800 1700 50  0000 C CNN
 	1    3800 1700
@@
 F 0 "C11" H 3010 1770 50  0000 L CNN
 F 1 "4.7u" H 3010 1620 50  0000 L CNN
-F 2 "Capacitors_Tantalum_SMD:TantalC_SizeA_EIA-3216_Wave" H 3000 1700 50  0001 C CNN
+F 2 "Capacitors_SMD:C_1206" H 3000 1700 50  0001 C CNN
 F 3 "" H 3000 1700 50  0000 C CNN
 	1    3000 1700
@@
 F 0 "C8" H 1410 6520 50  0000 L CNN
 F 1 "4.7u" H 1410 6370 50  0000 L CNN
-F 2 "Capacitors_Tantalum_SMD:TantalC_SizeA_EIA-3216_Wave" H 1400 6450 50  0001 C CNN
+F 2 "Capacitors_SMD:C_1206" H 1400 6450 50  0001 C CNN
 F 3 "" H 1400 6450 50  0000 C CNN
 	1    1400 6450
@@
 F 0 "C5" H 1010 6520 50  0000 L CNN
 F 1 "4.7u" H 1010 6370 50  0000 L CNN
-F 2 "Capacitors_Tantalum_SMD:TantalC_SizeA_EIA-3216_Wave" H 1000 6450 50  0001 C CNN
+F 2 "Capacitors_SMD:C_1206" H 1000 6450 50  0001 C CNN
 F 3 "" H 1000 6450 50  0000 C CNN
 	1    1000 6450

Commit message: rev 2.1.3 combine P1 and P2, update BOM, make R3 possible value
Parts:
- removed P1, P2: CONN_01X01, Pin_Headers:Pin_Header_Straight_1x01, symbol CONN_01X01
- added P1: CONN_01X02, Pin_Headers:Pin_Header_Straight_1x02, symbol CONN_01X02
- C22: value 100n -> dnp-100n
- P5: value CONN_01X02 -> dnp-CONN_01X02
- R16: value 1k -> dnp-1k
- R17, R18: value 3.9k -> dnp-3.9k
- R3: value 17k -> 20k
- R5: value DNP -> dnp-0
- U6: value AT24CS32-SSHM -> dnp-AT24CS32-SSHM
Connections:
- wire segments 263 -> 264
Changed lines of the file:
@@
 Title "Raspberry Pi Debugger"
 Date ""
-Rev "2.1.2"
+Rev "2.1.3"
 Comp "Carnegie Mellon University"
 Comment1 "Based on FT2232H Mini Module"
@@
 P 2200 6450
 F 0 "R3" H 2230 6470 50  0000 L CNN
-F 1 "17k" H 2230 6410 50  0000 L CNN
+F 1 "20k" H 2230 6410 50  0000 L CNN
 F 2 "Resistors_SMD:R_0603" H 2200 6450 50  0001 C CNN
 F 3 "" H 2200 6450 50  0000 C CNN
@@
 	1    0    0    -1
 $EndComp
-$Comp
-L CONN_01X01 P1
-U 1 1 56AA6C75
-P 4500 7150
-F 0 "P1" H 4500 7250 50  0000 C CNN
-F 1 "CONN_01X01" V 4600 7150 50  0000 C CNN
-F 2 "Pin_Headers:Pin_Header_Straight_1x01" H 4500 7150 50  0001 C CNN
-F 3 "" H 4500 7150 50  0000 C CNN
-	1    4500 7150
-	0    1    1    0
-$EndComp
 Wire Wire Line
 	4900 6350 5600 6350
 Text Label 5150 6350 0    60   ~ 0
 RPI_VBUS
-$Comp
-L CONN_01X01 P2
-U 1 1 56AA766C
-P 5000 7150
-F 0 "P2" H 5000 7250 50  0000 C CNN
-F 1 "CONN_01X01" V 5100 7150 50  0000 C CNN
-F 2 "Pin_Headers:Pin_Header_Straight_1x01" H 5000 7150 50  0001 C CNN
-F 3 "" H 5000 7150 50  0000 C CNN
-	1    5000 7150
-	0    1    1    0
-$EndComp
 Wire Wire Line
 	5000 6950 5000 6650
@@
 Connection ~ 5000 6350
 Wire Wire Line
-	4500 6950 4500 6650
+	4500 6650 4500 7050
 $Comp
 L R R5
@@
 P 3400 5850
 F 0 "R5" V 3480 5850 50  0000 C CNN
-F 1 "DNP" V 3400 5850 50  0000 C CNN
+F 1 "dnp-0" V 3400 5850 50  0000 C CNN
 F 2 "Resistors_SMD:R_0603" V 3330 5850 50  0001 C CNN
 F 3 "" H 3400 5850 50  0000 C CNN
@@
 P 8550 9250
 F 0 "U6" H 8350 9500 50  0000 C CNN
-F 1 "AT24CS32-SSHM" H 8900 8950 50  0000 C CNN
+F 1 "dnp-AT24CS32-SSHM" H 8900 8950 50  0000 C CNN
 F 2 "Housings_SSOP:TSSOP-8_4.4x3mm_Pitch0.65mm" H 9500 8850 50  0000 C CIN
 F 3 "" H 8550 9250 50  0000 C CNN
@@
 P 9050 9000
 F 0 "R17" H 9080 9020 50  0000 L CNN
-F 1 "3.9k" H 9080 8960 50  0000 L CNN
+F 1 "dnp-3.9k" H 9080 8960 50  0000 L CNN
 F 2 "Resistors_SMD:R_0603" H 9050 9000 50  0001 C CNN
 F 3 "" H 9050 9000 50  0000 C CNN
@@
 P 9450 9000
 F 0 "R18" H 9480 9020 50  0000 L CNN
-F 1 "3.9k" H 9480 8960 50  0000 L CNN
+F 1 "dnp-3.9k" H 9480 8960 50  0000 L CNN
 F 2 "Resistors_SMD:R_0603" H 9450 9000 50  0001 C CNN
 F 3 "" H 9450 9000 50  0000 C CNN
@@
 P 7850 9000
 F 0 "R16" H 7880 9020 50  0000 L CNN
-F 1 "1k" H 7880 8960 50  0000 L CNN
+F 1 "dnp-1k" H 7880 8960 50  0000 L CNN
 F 2 "Resistors_SMD:R_0603" H 7850 9000 50  0001 C CNN
 F 3 "" H 7850 9000 50  0000 C CNN
@@
 P 7550 9500
 F 0 "P5" H 7550 9650 50  0000 C CNN
-F 1 "CONN_01X02" V 7650 9500 50  0000 C CNN
+F 1 "dnp-CONN_01X02" V 7650 9500 50  0000 C CNN
 F 2 "Pin_Headers:Pin_Header_Straight_1x02" H 7550 9500 50  0001 C CNN
 F 3 "" H 7550 9500 50  0000 C CNN
@@
 P 7050 9000
 F 0 "C22" H 7060 9070 50  0000 L CNN
-F 1 "100n" H 7060 8920 50  0000 L CNN
+F 1 "dnp-100n" H 7060 8920 50  0000 L CNN
 F 2 "Capacitors_SMD:C_0603" H 7050 9000 50  0001 C CNN
 F 3 "" H 7050 9000 50  0000 C CNN
@@
 	4100 6450 4100 6350
 Connection ~ 4100 6350
+$Comp
+L CONN_01X02 P1
+U 1 1 5785F2B0
+P 5200 7000
+F 0 "P1" H 5200 7150 50  0000 C CNN
+F 1 "CONN_01X02" V 5300 7000 50  0000 C CNN
+F 2 "Pin_Headers:Pin_Header_Straight_1x02" H 5200 7000 50  0001 C CNN
+F 3 "" H 5200 7000 50  0000 C CNN
+	1    5200 7000
+	1    0    0    1
+$EndComp
+Wire Wire Line
+	4500 7050 5000 7050
 $EndSCHEMATC

Commit message: change shunt resistor to 0.05 ohm
Parts:
- R7: value 0.01 -> 0.05
Changed lines of the file:
@@
 P 4750 6350
 F 0 "R7" V 4830 6350 50  0000 C CNN
-F 1 "0.01" V 4750 6350 50  0000 C CNN
+F 1 "0.05" V 4750 6350 50  0000 C CNN
 F 2 "Resistors_SMD:R_1206" V 4680 6350 50  0001 C CNN
 F 3 "" H 4750 6350 50  0000 C CNN

Commit message: swap rpi connector for no paste verison and no stuff
Parts:
- P4: value CONN_02X20 -> dnp-REF-182665-01; footprint debugger2-special:Pin_Header_Straight_TH-SMT_2x20 -> debugger2-special:Pin_Header_Straight_TH-SMT-NoPaste_2x20
Changed lines of the file:
@@
 P 9450 2100
 F 0 "P4" H 9450 3150 50  0000 C CNN
-F 1 "CONN_02X20" V 9450 2100 50  0000 C CNN
-F 2 "debugger2-special:Pin_Header_Straight_TH-SMT_2x20" H 9450 1150 50  0001 C CNN
+F 1 "dnp-REF-182665-01" V 9450 2100 50  0000 C CNN
+F 2 "debugger2-special:Pin_Header_Straight_TH-SMT-NoPaste_2x20" H 9450 1150 50  0001 C CNN
 F 3 "" H 9450 1150 50  0000 C CNN
 	1    9450 2100

Commit message: update U2 and U3 part no on bom and schematic. prevents U2 smoking
Parts:
- U2: value MIC9409x_SC-70 -> MIC94092_SC-70
- U3: value FT2232H -> FT2232HL
Changed lines of the file:
@@
 P 5900 3100
 F 0 "U3" H 5350 5300 60  0000 C CNN
-F 1 "FT2232H" H 5500 1100 60  0000 C CNN
+F 1 "FT2232HL" H 5500 1100 60  0000 C CNN
 F 2 "Housings_QFP:TQFP-64_10x10mm_Pitch0.5mm" H 4900 3950 60  0001 C CNN
 F 3 "" H 4900 3950 60  0000 C CNN
@@
 P 3400 6500
 F 0 "U2" H 3150 6850 60  0000 L CNN
-F 1 "MIC9409x_SC-70" H 3000 6150 60  0000 L CNN
+F 1 "MIC94092_SC-70" H 3000 6150 60  0000 L CNN
 F 2 "TO_SOT_Packages_SMD:SC-70-6" H 3400 6500 60  0001 C CNN
 F 3 "" H 3400 6500 60  0000 C CNN
